File: UNOQ_ExperimentalShield/UNOQ_ExperimentalShield.kicad_pcb (KiCad board)
At the start: 4 copper layers, 68.6 x 53.3 mm, 128 parts, among them CN1 485, CN2 USB, CN3 Can, CN4 Can, CN5 485, J1 Power, J2 Digital/PWM, J3 Analog, J4 Digital/PWM, SW1 Usr1, SW2 Usr1, SW3 Usr1, SW4 Usr1, U1 25LCxxx, U2 TMP102xxDRL, U3 MAX3485ESA-MS, U4 CH340N, U5 TJA1051T-3

Commit message: List of changes/fixes: - Buttons reducto 2 and moved to A2, A3 - Fixed TX/RX CAN lines for R4 - Buttons tied to Vio - Pots tied to Vio - Added ATECC608 secure element
Parts:
- removed the G*** at (165.5, 70.6)
- removed R11, R12: 10k, Resistor_SMD:R_0402_1005Metric
- removed SW3, SW4: Usr1, Button_Switch_SMD:SW_SPST_PTS810
- removed kibuzzard-69595BF0: G***, kibuzzard-69595BF0
- removed kibuzzard-69595BF8: G***, kibuzzard-69595BF8
- removed kibuzzard-695F89C6: G***, kibuzzard-695F89C6
- removed kibuzzard-697C8A8B: G***, kibuzzard-697C8A8B
- removed kibuzzard-697C8A92: G***, kibuzzard-697C8A92
- added C7: 100nF, Capacitor_SMD:C_0402_1005Metric, F.Cu at (166.3, 67.8)
- added U7: ATECC608A-SSHDA, Package_SO:SOIC-8_3.9x4.9mm_P1.27mm, F.Cu at (164.0, 71.2)
- added kibuzzard-69DFD334: G***, kibuzzard-69DFD334, F.Cu at (167.2, 87.4)
- added kibuzzard-69E2216E: G***, kibuzzard-69E2216E, F.Cu at (152.8, 67.9)
- added kibuzzard-69E22173: G***, kibuzzard-69E22173, F.Cu at (152.8, 74.6)
- added kibuzzard-69E66319: G***, kibuzzard-69E66319, F.Cu at (162.8, 67.5)
- moved SW2 7.96 mm to (156.7, 74.7)
- moved SW1 6.63 mm to (156.7, 67.9)
- moved R10 5.98 mm to (158.7, 72.1), turned to 0 degrees
- moved kibuzzard-6987894B 5.36 mm to (106.0, 90.2), turned to 0 degrees
- moved R9 4.82 mm to (158.7, 65.3), turned to 0 degrees
- moved G*** 0.46 mm to (103.9, 86.1)
Connections:
- J2 pad 5: /D13/SCK/CANTX -> /D13/SCK/CANRX
- J2 pad 8: /D10/CS/CANRX -> /D10/CS/CANTX
- JP1 pad 2: /D13/SCK/CANTX -> /D10/CS/CANTX
- JP1 pad 3: /SCK -> /CS
- JP2 pad 2: /D10/CS/CANRX -> /D13/SCK/CANRX
- JP2 pad 3: /CS -> /SCK
- R10 pad 1: +3V3 -> /Vio
- R10 pad 2: /D3* -> /A3
- R9 pad 1: +3V3 -> /Vio
- R9 pad 2: /D2 -> /A2
- RV1 pad 1: +3V3 -> /Vio
- RV2 pad 1: +3V3 -> /Vio
- SW1 pad 2: /D2 -> /A2
- SW2 pad 2: /D3* -> /A3
Routing:
- net /D13/SCK/CANTX: track 75.4 -> 0.00 mm
- net /D13/SCK/CANRX: track 0.00 -> 71.0 mm
- net /D10/CS/CANTX: track 0.00 -> 70.7 mm
- net /D10/CS/CANRX: track 65.3 -> 0.00 mm
- net /A2: track 0.00 -> 49.9 mm, vias 0 -> 2
- net /Vio: track 94.4 -> 141.5 mm, vias 11 -> 16
- net /A3: track 0.00 -> 41.1 mm, vias 0 -> 2
- net /D7: track 39.5 -> 8.94 mm
- net /D6*: track 34.1 -> 9.04 mm
- net /D3*: track 26.2 -> 4.86 mm
- net +3V3: track 229.9 -> 218.1 mm, vias 16 -> 12
- net /SDA/A4: track 76.8 -> 85.9 mm
- net /SCL/A5: track 74.5 -> 82.9 mm
- net /CS: track 74.5 -> 80.1 mm
- net /D2: track 72.3 -> 67.0 mm
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