File: UNOQ_ExperimentalShield/UNOQ_ExperimentalShield.kicad_sch (KiCad schematic)
At the start: 74 parts, among them CN1 485, CN2 USB, CN3 Can, CN4 Can, CN5 485, J1 Power, J2 Digital/PWM, J3 Analog, J4 Digital/PWM, SW1 Usr1, SW2 Usr1, SW3 Usr1, SW4 Usr1, U1 25LCxxx, U2 TMP102xxDRL, U3 MAX3485ESA-MS, U4 CH340N, U5 TJA1051T-3

Commit message: List of changes/fixes: - Buttons reducto 2 and moved to A2, A3 - Fixed TX/RX CAN lines for R4 - Buttons tied to Vio - Pots tied to Vio - Added ATECC608 secure element
Parts:
- removed R11, R12: 10k, Resistor_SMD:R_0402_1005Metric, symbol Device:R
- removed SW3, SW4: Usr1, Button_Switch_SMD:SW_SPST_PTS810, symbol Switch:SW_Push
- added C7: 100nF, Capacitor_SMD:C_0402_1005Metric, symbol Device:C
- added U7: ATECC608A-SSHDA, Package_SO:SOIC-8_3.9x4.9mm_P1.27mm, symbol Security:ATECC608A-SSHDA
Connections:
- net +3V3: now also C7.1, U7.8 (VCC); no longer R10.1, R9.1, RV1.1, RV2.1
- net A2: now also R9.2, SW1.2
- net A3: now also R10.2, SW2.2
- net CS: now also JP1.3 (B); no longer JP2.3 (B)
- net D2: no longer R9.2, SW1.2
- net D3*: no longer R10.2, SW2.2
- net GND: now also C7.2, U7.4 (GND)
- net SCK: now also JP2.3 (B); no longer JP1.3 (B)
- net SCL/A5: now also U7.6 (SCL)
- net SDA/A4: now also U7.5 (SDA)
- net Vio: now also R10.1, R9.1, RV1.1, RV2.1
- net D10/CS/CANRX renamed D10/CS/CANTX
- net D10/CS/CANTX: now also JP1.2 (C); no longer JP2.2 (C)
- net D13/SCK/CANTX renamed D13/SCK/CANRX
- net D13/SCK/CANRX: now also JP2.2 (C); no longer JP1.2 (C)
Other:
- moved on the sheet: R10, R9, SW1, SW2
